Commit message: aded color materials

File: src/robot_description/urdf/agrobot_v2_core.xacro (robot description, xacro)
@@ -1,4 +1,5 @@
 <?xml version="1.0"?>
 <robot xmlns:xacro="http://www.ros.org/wiki/xacro" name="robot_description">
+  <xacro:include filename="material.xacro" />
   <link name="base_link">
     <inertial>
@@ -24,9 +25,5 @@
           filename="package://robot_description/meshes/base_link.STL" />
       </geometry>
-      <material
-        name="">
-        <color
-          rgba="0.79216 0.81961 0.93333 1" />
-      </material>
+      <material name="slate_blue" />
     </visual>
     <collision>
@@ -63,9 +60,5 @@
           filename="package://robot_description/meshes/lidar_link.STL" />
       </geometry>
-      <material
-        name="">
-        <color
-          rgba="0.75294 0.75294 0.75294 0.4" />
-      </material>
+      <material name="deep_ocean_blue" />
     </visual>
     <collision>
@@ -114,9 +107,5 @@
           filename="package://robot_description/meshes/right_wheel_link.STL" />
       </geometry>
-      <material
-        name="">
-        <color
-          rgba="0.75294 0.75294 0.75294 1" />
-      </material>
+      <material name="dark_teal"/>
     </visual>
     <collision>
@@ -171,9 +160,5 @@
           filename="package://robot_description/meshes/left_wheel_link.STL" />
       </geometry>
-      <material
-        name="">
-        <color
-          rgba="0.75294 0.75294 0.75294 1" />
-      </material>
+      <material name="dark_teal"/>
     </visual>
     <collision>
@@ -228,9 +213,5 @@
           filename="package://robot_description/meshes/castor_l_swivel_link.STL" />
       </geometry>
-      <material
-        name="">
-        <color
-          rgba="0.89804 0.91765 0.92941 1" />
-      </material>
+      <material name="slate_blue"/>
     </visual>
     <collision>
@@ -285,9 +266,5 @@
           filename="package://robot_description/meshes/castor_l_wheel_link.STL" />
       </geometry>
-      <material
-        name="">
-        <color
-          rgba="0.89804 0.91765 0.92941 1" />
-      </material>
+      <material name="dark_teal"/>
     </visual>
     <collision>
@@ -342,9 +319,5 @@
           filename="package://robot_description/meshes/castor_r_swivel_link.STL" />
       </geometry>
-      <material
-        name="">
-        <color
-          rgba="0.89804 0.91765 0.92941 1" />
-      </material>
+      <material name="slate_blue"/>
     </visual>
     <collision>
@@ -399,9 +372,5 @@
           filename="package://robot_description/meshes/castor_r_wheel_link.STL" />
       </geometry>
-      <material
-        name="">
-        <color
-          rgba="0.89804 0.91765 0.92941 1" />
-      </material>
+      <material name="dark_teal"/>
     </visual>
     <collision>
@@ -456,9 +425,5 @@
           filename="package://robot_description/meshes/arm_base_link.STL" />
       </geometry>
-      <material
-        name="">
-        <color
-          rgba="0.2 0.2 0.2 1" />
-      </material>
+      <material name="dark_teal"/>
     </visual>
     <collision>
@@ -507,9 +472,5 @@
           filename="package://robot_description/meshes/base_yaw_link.STL" />
       </geometry>
-      <material
-        name="">
-        <color
-          rgba="0.98824 0.73725 0.51765 1" />
-      </material>
+      <material name="industrial_orange"/>
     </visual>
     <collision>
@@ -566,9 +527,5 @@
           filename="package://robot_description/meshes/shoulder_link.STL" />
       </geometry>
-      <material
-        name="">
-        <color
-          rgba="0.98824 0.73725 0.51765 1" />
-      </material>
+      <material name="industrial_orange"/>
     </visual>
     <collision>
@@ -625,9 +582,5 @@
           filename="package://robot_description/meshes/elbow_link.STL" />
       </geometry>
-      <material
-        name="">
-        <color
-          rgba="0.98824 0.73725 0.51765 1" />
-      </material>
+      <material name="industrial_orange"/>
     </visual>
     <collision>
@@ -684,9 +637,5 @@
           filename="package://robot_description/meshes/wrist_pitch_link.STL" />
       </geometry>
-      <material
-        name="">
-        <color
-          rgba="0.98824 0.73725 0.51765 1" />
-      </material>
+      <material name="industrial_orange"/>
     </visual>
     <collision>
@@ -743,9 +692,5 @@
           filename="package://robot_description/meshes/wrist_roll_link.STL" />
       </geometry>
-      <material
-        name="">
-        <color
-          rgba="0.98824 0.73725 0.51765 1" />
-      </material>
+      <material name="sandy_yellow"/>
     </visual>
     <collision>

Commit message: added camera link

File: src/robot_description/urdf/agrobot_v2_core.xacro (robot description, xacro)
@@ -707,5 +707,5 @@
     type="revolute">
     <origin
-      xyz="0.081369 0.054095 -0.0075371"
+      xyz="0.081369 0.054095 0"
       rpy="0 0 0" />
     <parent
@@ -724,3 +724,27 @@
       friction="0.1" />
   </joint>
+<link name="camera_link">
+    <visual>
+      <origin xyz="0 0 0" rpy="0 0 0"/>
+      <geometry>
+        <box size="0.01 0.01 0.01"/>
+      </geometry>
+      <material name="deep_ocean_blue"/>
+    </visual>
+    <collision>
+      <origin xyz="0 0 0" rpy="0 0 0"/>
+      <geometry>
+        <box size="0.01 0.01 0.01"/>
+      </geometry>
+    </collision>
+    <inertial>
+      <mass value="0.01"/>
+      <inertia ixx="1e-6" ixy="0" ixz="0" iyy="1e-6" iyz="0" izz="1e-6"/>
+    </inertial>
+  </link>
+  <joint name="camera_joint" type="fixed">
+    <origin xyz="0.04 0.0 0" rpy="0 0 0" />
+    <parent link="wrist_roll_link" />
+    <child link="camera_link" />
+  </joint>
 </robot>

Commit message: added dummy for the camera lens ; since the axes of the stander robot and the axes for image processing libraries are different

File: src/robot_description/urdf/agrobot_v2_core.xacro (robot description, xacro)
@@ -747,3 +747,9 @@
     <child link="camera_link" />
   </joint>
+  <link name="camera_depth_optical_frame"/>
+  <joint name="camera_optical_joint" type="fixed">
+    <origin xyz="0 0 0" rpy="-1.5708 0 -1.5708" />
+    <parent link="camera_link" />
+    <child link="camera_depth_optical_frame" />
+  </joint>
 </robot>

Commit message: added base footprint link and joint, updated material attributes for various links

File: src/robot_description/urdf/agrobot_v2_core.xacro (robot description, xacro)
@@ -1,4 +1,10 @@
 <?xml version="1.0"?>
 <robot xmlns:xacro="http://www.ros.org/wiki/xacro" name="robot_description">
+  <link name="base_footprint" />
+  <joint name="base_footprint_joint" type="fixed">
+    <parent link="base_footprint" />
+    <child link="base_link" />
+    <origin xyz="0 0 0" rpy="0 0 0" />
+  </joint>
   <link name="base_link">
     <inertial>
@@ -106,5 +112,5 @@
           filename="package://robot_description/meshes/right_wheel_link.STL" />
       </geometry>
-      <material name="dark_teal"/>
+      <material name="dark_teal" />
     </visual>
     <collision>
@@ -130,6 +136,6 @@
       xyz="0 0 1" />
     <limit
-      effort="10"
-      velocity="10" />
+      effort="500"
+      velocity="20" />
     <dynamics
       damping="0.1"
@@ -159,5 +165,5 @@
           filename="package://robot_description/meshes/left_wheel_link.STL" />
       </geometry>
-      <material name="dark_teal"/>
+      <material name="dark_teal" />
     </visual>
     <collision>
@@ -183,6 +189,6 @@
       xyz="0 0 1" />
     <limit
-      effort="10"
-      velocity="10" />
+      effort="500"
+      velocity="20" />
     <dynamics
       damping="0.1"
@@ -212,5 +218,5 @@
           filename="package://robot_description/meshes/castor_l_swivel_link.STL" />
       </geometry>
-      <material name="slate_blue"/>
+      <material name="slate_blue" />
     </visual>
     <collision>
@@ -265,5 +271,5 @@
           filename="package://robot_description/meshes/castor_l_wheel_link.STL" />
       </geometry>
-      <material name="dark_teal"/>
+      <material name="dark_teal" />
     </visual>
     <collision>
@@ -318,5 +324,5 @@
           filename="package://robot_description/meshes/castor_r_swivel_link.STL" />
       </geometry>
-      <material name="slate_blue"/>
+      <material name="slate_blue" />
     </visual>
     <collision>
@@ -371,5 +377,5 @@
           filename="package://robot_description/meshes/castor_r_wheel_link.STL" />
       </geometry>
-      <material name="dark_teal"/>
+      <material name="dark_teal" />
     </visual>
     <collision>
@@ -424,5 +430,5 @@
           filename="package://robot_description/meshes/arm_base_link.STL" />
       </geometry>
-      <material name="dark_teal"/>
+      <material name="dark_teal" />
     </visual>
     <collision>
@@ -471,5 +477,5 @@
           filename="package://robot_description/meshes/base_yaw_link.STL" />
       </geometry>
-      <material name="industrial_orange"/>
+      <material name="industrial_orange" />
     </visual>
     <collision>
@@ -526,5 +532,5 @@
           filename="package://robot_description/meshes/shoulder_link.STL" />
       </geometry>
-      <material name="industrial_orange"/>
+      <material name="industrial_orange" />
     </visual>
     <collision>
@@ -581,5 +587,5 @@
           filename="package://robot_description/meshes/elbow_link.STL" />
       </geometry>
-      <material name="industrial_orange"/>
+      <material name="industrial_orange" />
     </visual>
     <collision>
@@ -636,5 +642,5 @@
           filename="package://robot_description/meshes/wrist_pitch_link.STL" />
       </geometry>
-      <material name="industrial_orange"/>
+      <material name="industrial_orange" />
     </visual>
     <collision>
@@ -691,5 +697,5 @@
           filename="package://robot_description/meshes/wrist_roll_link.STL" />
       </geometry>
-      <material name="sandy_yellow"/>
+      <material name="sandy_yellow" />
     </visual>
     <collision>
@@ -723,21 +729,21 @@
       friction="0.1" />
   </joint>
-<link name="camera_link">
-    <visual>
-      <origin xyz="0 0 0" rpy="0 0 0"/>
-      <geometry>
-        <box size="0.01 0.01 0.01"/>
-      </geometry>
-      <material name="deep_ocean_blue"/>
-    </visual>
-    <collision>
-      <origin xyz="0 0 0" rpy="0 0 0"/>
-      <geometry>
-        <box size="0.01 0.01 0.01"/>
-      </geometry>
-    </collision>
-    <inertial>
-      <mass value="0.01"/>
-      <inertia ixx="1e-6" ixy="0" ixz="0" iyy="1e-6" iyz="0" izz="1e-6"/>
+  <link name="camera_link">
+    <visual>
+      <origin xyz="0 0 0" rpy="0 0 0" />
+      <geometry>
+        <box size="0.01 0.01 0.01" />
+      </geometry>
+      <material name="deep_ocean_blue" />
+    </visual>
+    <collision>
+      <origin xyz="0 0 0" rpy="0 0 0" />
+      <geometry>
+        <box size="0.01 0.01 0.01" />
+      </geometry>
+    </collision>
+    <inertial>
+      <mass value="0.01" />
+      <inertia ixx="1e-6" ixy="0" ixz="0" iyy="1e-6" iyz="0" izz="1e-6" />
     </inertial>
   </link>
@@ -747,5 +753,5 @@
     <child link="camera_link" />
   </joint>
-  <link name="camera_depth_optical_frame"/>
+  <link name="camera_depth_optical_frame" />
   <joint name="camera_optical_joint" type="fixed">
     <origin xyz="0 0 0" rpy="-1.5708 0 -1.5708" />
